File: GPIO HAT 1/GPIO HAT 1/GPIO HAT 1.kicad_pcb (KiCad board)
At the start: 4 copper layers, 68 x 85 mm, 69 parts, among them J1 Conn_01x05, J10 Conn_01x05, J11 Conn_01x05, J12 Conn_01x05, J13 Conn_01x05, J14 Conn_01x05, J15 Conn_01x05, J16 Conn_01x05, J17 Conn_01x05, J18 Conn_01x05, J19 Conn_01x05, J2 Conn_01x05, J20 Conn_01x05, J23 2.54-2*20PPC104, J24 2.54-2*20PPC104, J3 Conn_01x05, J4 Conn_01x05, J5 Conn_01x05, J6 Conn_01x05, J7 Conn_01x05, J8 Conn_01x05, J9 Conn_01x05, U1 TXB0108DQSR, U10 TXB0108DQSR, U2 TXB0108DQSR, U3 TXB0108DQSR, U4 TXB0108DQSR, U5 TXB0108DQSR, U6 TXB0108DQSR, U7 TXB0108DQSR, U8 TXB0108DQSR, U9 TXB0108DQSR

Commit message: Update
Gerber Generated
Other:
- board text added: "Designed in Gujarat,India."
- board text added: "R0.1"
- board text added: "V1.0"
- board text removed: "VERSION 1.0"
