File: GPIO HAT 2/GPIO HAT 2/GPIO HAT 2.kicad_sch (KiCad schematic)
At the start: 99 parts, among them J1 ., J10 ., J11 ., J12 ., J13 ., J14 ., J15 ., J16 ., J17 ., J18 ., J19 ., J2 ., J20 ., J21 LVDS, J22 LVDS, J23 02x02, J24 USB_C_Receptacle_PowerOnly_6P, J3 ., J4 ., J5 ., J6 ., J7 ., J8 ., J9 ., U1 TXB0108DQSR, U10 TXB0108DQSR, U12 SY8088IAAC, U13 SY8088IAAC, U14 TPS2117, U2 TXB0108DQSR, U3 TXB0108DQSR, U4 TXB0108DQSR, U5 TXB0108DQSR, U6 TXB0108DQSR, U7 TXB0108DQSR, U8 TXB0108DQSR, U9 TXB0108DQSR

Commit message: Update
Gerber Generated
Parts:
- renumbered C2 to C1, C44 to C10, C43 to C11, C16 to C12, C17 to C13, C18 to C14, C19 to C15, C20 to C16, C21 to C17, C22 to C18, C24 to C19, C3 to C2, C26 to C20, C28 to C21, C34 to C22, C36 to C23, C38 to C24, C23 to C25, C25 to C26, C33 to C28, C35 to C29, C4 to C3, C37 to C30, C30 to C31, C40 to C33, C42 to C34, C29 to C35, C31 to C36, C39 to C37, C41 to C38, C5 to C4, C6 to C5, C7 to C6, C8 to C7, C1 to C8, J24 to J1, J15 to J10, J2 to J11, J4 to J12, J6 to J13, J12 to J14, J14 to J15, J7 to J17, J9 to J18, J17 to J19, J23 to J2, J19 to J20, J8 to J21, J10 to J22, J18 to J23, J20 to J24, J22 to J3, J21 to J4, J1 to J5, J3 to J6, J5 to J7, J11 to J8, J13 to J9, JM2 to JM1, JM4 to JM2, JM1 to JM3, JM3 to JM4, L3 to L2, R16 to R1, R3 to R10, R6 to R11, R7 to R12, R8 to R13, R4 to R14, R5 to R15, R9 to R16, R10 to R17, R17 to R2, R20 to R3, R22 to R4, R21 to R5, R18 to R6, R19 to R7, R1 to R8, R2 to R9, U12 to U1, U4 to U10, U5 to U11, U9 to U12, U10 to U13, U14 to U2, U13 to U3, U1 to U4, U2 to U5, U3 to U6, U6 to U7, U7 to U8, U8 to U9

Commit message: GPIO number change, CC1 & CC2 tied to GND
Parts:
- removed U11, U12, U13: TXB0108DQSR, VAAMAN2:TXB0108DQSR, symbol VAAMAN2:TXB0108DQSR
- removed U2: TPS2117, VAAMAN2:TPS2117, symbol VAAMAN2:TPS2117
- added R18, R19: 5.1K, VAAMAN2:0402_Res, symbol Device:R_US
- added U1, U2, U3: ~, symbol VAAMAN2:TXB0108DQSR
- added U13: TPS2117, VAAMAN2:TPS2117, symbol VAAMAN2:TPS2117
- J23: renamed from J1; Manufacturer Part Number (none) -> U262-061N-4BVC10
- L1, L2: Manufacturer Part Number (none) -> GCNR4030-3R3NC
- U10, U4, U5, U6, U7, U8, U9: value TXB0108DQSR -> ~; footprint VAAMAN2:TXB0108DQSR -> (none); CASE/PACKAGE USON-20 -> (none); Manufacturer Part Number (none) -> TXB0108DQSR; Vicharak-PN (none) -> V001766
- U11: renamed from U1; Manufacturer Part Number (none) -> SY8088IAAC; Vicharak-PN (none) -> V001502
- U12: renamed from U3; Manufacturer Part Number (none) -> SY8088IAAC; Vicharak-PN (none) -> V001502
- renumbered J5 to J1, J22 to J10, J8 to J11, J14 to J12, J9 to J13, J15 to J14, J10 to J15, J19 to J17, J23 to J18, J20 to J19, J11 to J2, J24 to J20, J4 to J21, J3 to J22, J2 to J24, J6 to J3, J12 to J4, J7 to J5, J13 to J6, J17 to J7, J21 to J8, J18 to J9
Connections:
- net 3.3V: now also U1.16 (VCCB), U2.16 (VCCB), U3.16 (VCCB)
- net 5V: now also U13.2 (VOUT), U13.7 (VOUT)
- net 5V_1: now also U13.3 (VIN1), U13.5 (MODE); no longer J23.B9 (VBUS)
- net GND: now also R18.2, R19.2, U1.15 (GND), U13.1 (GND), U2.15 (GND), U3.15 (GND)
- net GPIOB_TXN00: now also U3.17 (B4); no longer U7.17 (B4)
- net GPIOB_TXN01: now also U3.19 (B2); no longer U7.19 (B2)
- net GPIOB_TXN02: now also U3.13 (B6); no longer U7.13 (B6)
- net GPIOB_TXN03: now also U4.14 (B5); no longer U8.14 (B5)
- net GPIOB_TXN04: now also U4.18 (B3); no longer U8.18 (B3)
- net GPIOB_TXN05: now also U4.11 (B8); no longer U8.11 (B8)
- net GPIOB_TXN06: now also U4.19 (B2); no longer U8.19 (B2)
- net GPIOB_TXN09: now also U5.12 (B7)
- net GPIOB_TXN10: now also U5.13 (B6)
- net GPIOB_TXN12: now also U5.20 (B1)
- net GPIOB_TXN13: now also U3.11 (B8); no longer U7.11 (B8)
- net GPIOB_TXN14: now also U10.17 (B4)
- net GPIOB_TXN16: now also U10.13 (B6)
- net GPIOB_TXN17: now also U10.11 (B8)
- net GPIOB_TXN18: now also U5.17 (B4)
- net GPIOB_TXN19: now also U10.19 (B2)
- net GPIOB_TXP00: now also U3.18 (B3); no longer U7.18 (B3)
- net GPIOB_TXP01: now also U3.20 (B1); no longer U7.20 (B1)
- net GPIOB_TXP02: now also U3.14 (B5); no longer U7.14 (B5)
- net GPIOB_TXP03: now also U4.13 (B6); no longer U8.13 (B6)
- net GPIOB_TXP04: now also U4.17 (B4); no longer U8.17 (B4)
- net GPIOB_TXP05: now also U4.12 (B7); no longer U8.12 (B7)
- net GPIOB_TXP06: now also U4.20 (B1); no longer U8.20 (B1)
- net GPIOB_TXP09: now also U5.11 (B8)
- net GPIOB_TXP10: now also U5.14 (B5)
- net GPIOB_TXP12: now also U5.19 (B2)
- net GPIOB_TXP13: now also U3.12 (B7); no longer U7.12 (B7)
- net GPIOB_TXP14: now also U10.18 (B3)
- net GPIOB_TXP16: now also U10.14 (B5)
- net GPIOB_TXP17: now also U10.12 (B7)
- net GPIOB_TXP18: now also U5.18 (B3)
- net GPIOB_TXP19: now also U10.20 (B1)
- net GPIOB__TXN00: now also U3.4 (A4); no longer U7.4 (A4)
- net GPIOB__TXN01: now also U3.2 (A2); no longer U7.2 (A2)
- net GPIOB__TXN02: now also U3.8 (A6); no longer U7.8 (A6)
- net GPIOB__TXN03: now also U4.7 (A5); no longer U8.7 (A5)
- net GPIOB__TXN04: now also U4.3 (A3); no longer U8.3 (A3)
- net GPIOB__TXN05: now also U4.10 (A8); no longer U8.10 (A8)
- net GPIOB__TXN06: now also U4.2 (A2); no longer U8.2 (A2)
- net GPIOB__TXN09: now also U5.9 (A7)
- net GPIOB__TXN10: now also U5.8 (A6)
- net GPIOB__TXN12: now also U5.1 (A1)
- net GPIOB__TXN13: now also U3.10 (A8); no longer U7.10 (A8)
- net GPIOB__TXN14: now also U10.4 (A4)
- net GPIOB__TXN16: now also U10.8 (A6)
- net GPIOB__TXN17: now also U10.10 (A8)
- net GPIOB__TXN18: now also U5.4 (A4)
- net GPIOB__TXN19: now also U10.2 (A2)
- net GPIOB__TXP00: now also U3.3 (A3); no longer U7.3 (A3)
- net GPIOB__TXP01: now also U3.1 (A1); no longer U7.1 (A1)
- net GPIOB__TXP02: now also U3.7 (A5); no longer U7.7 (A5)
- net GPIOB__TXP03: now also U4.8 (A6); no longer U8.8 (A6)
- net GPIOB__TXP04: now also U4.4 (A4); no longer U8.4 (A4)
- net GPIOB__TXP05: now also U4.9 (A7); no longer U8.9 (A7)
- net GPIOB__TXP06: now also U4.1 (A1); no longer U8.1 (A1)
- net GPIOB__TXP09: now also U5.10 (A8)
- net GPIOB__TXP10: now also U5.7 (A5)
- net GPIOB__TXP12: now also U5.2 (A2)
- net GPIOB__TXP13: now also U3.9 (A7); no longer U7.9 (A7)
- net GPIOB__TXP14: now also U10.3 (A3)
- net GPIOB__TXP16: now also U10.7 (A5)
- net GPIOB__TXP17: now also U10.9 (A7)
- net GPIOB__TXP18: now also U5.3 (A3)
- net GPIOB__TXP19: now also U10.1 (A1)
- net GPIOT_RXN01: now also U1.13 (B6); no longer U5.13 (B6)
- net GPIOT_RXN02: now also U7.14 (B5); no longer U6.14 (B5)
- net GPIOT_RXN03: now also U6.12 (B7); no longer U4.12 (B7)
- net GPIOT_RXN04: now also U7.18 (B3); no longer U6.18 (B3)
- net GPIOT_RXN05: now also U1.18 (B3); no longer U5.18 (B3)
- net GPIOT_RXN06: now also U1.12 (B7); no longer U5.12 (B7)
- net GPIOT_RXN07: now also U7.20 (B1); no longer U6.20 (B1)
- net GPIOT_RXN08: now also U6.14 (B5); no longer U4.14 (B5)
- net GPIOT_RXN09: now also U2.18 (B3); no longer U10.18 (B3)
- net GPIOT_RXN11: now also U8.18 (B3)
- net GPIOT_RXN12: now also U8.12 (B7)
- net GPIOT_RXN13: now also U8.19 (B2)
- net GPIOT_RXN14: now also U8.14 (B5)
- net GPIOT_RXN15: now also U2.12 (B7); no longer U10.12 (B7)
- net GPIOT_RXN16: now also U2.14 (B5); no longer U10.14 (B5)
- net GPIOT_RXN17: now also U2.19 (B2); no longer U10.19 (B2)
- net GPIOT_RXN18: now also U6.20 (B1); no longer U4.20 (B1)
- net GPIOT_RXN19: now also U7.12 (B7); no longer U6.12 (B7)
- net GPIOT_RXN20: now also U1.19 (B2); no longer U5.19 (B2)
- net GPIOT_RXN21: now also U6.17 (B4); no longer U4.17 (B4)
- net GPIOT_RXP01: now also U1.14 (B5); no longer U5.14 (B5)
- net GPIOT_RXP02: now also U7.13 (B6); no longer U6.13 (B6)
- net GPIOT_RXP03: now also U6.11 (B8); no longer U4.11 (B8)
- net GPIOT_RXP04: now also U7.17 (B4); no longer U6.17 (B4)
- net GPIOT_RXP05: now also U1.17 (B4); no longer U5.17 (B4)
- net GPIOT_RXP06: now also U1.11 (B8); no longer U5.11 (B8)
- net GPIOT_RXP07: now also U7.19 (B2); no longer U6.19 (B2)
- net GPIOT_RXP08: now also U6.13 (B6); no longer U4.13 (B6)
- net GPIOT_RXP09: now also U2.17 (B4); no longer U10.17 (B4)
- net GPIOT_RXP11: now also U8.17 (B4)
- net GPIOT_RXP12: now also U8.11 (B8)
- net GPIOT_RXP13: now also U8.20 (B1)
- net GPIOT_RXP14: now also U8.13 (B6)
- net GPIOT_RXP15: now also U2.11 (B8); no longer U10.11 (B8)
- net GPIOT_RXP16: now also U2.13 (B6); no longer U10.13 (B6)
- net GPIOT_RXP17: now also U2.20 (B1); no longer U10.20 (B1)
- net GPIOT_RXP18: now also U6.19 (B2); no longer U4.19 (B2)
- net GPIOT_RXP19: now also U7.11 (B8); no longer U6.11 (B8)
- net GPIOT_RXP20: now also U1.20 (B1); no longer U5.20 (B1)
- net GPIOT_RXP21: now also U6.18 (B3); no longer U4.18 (B3)
- net GPIOT__RXN01: now also U1.8 (A6); no longer U5.8 (A6)
- net GPIOT__RXN02: now also U7.7 (A5); no longer U6.7 (A5)
- net GPIOT__RXN03: now also U6.9 (A7); no longer U4.9 (A7)
- net GPIOT__RXN04: now also U7.3 (A3); no longer U6.3 (A3)
- net GPIOT__RXN05: now also U1.3 (A3); no longer U5.3 (A3)
- net GPIOT__RXN06: now also U1.9 (A7); no longer U5.9 (A7)
- net GPIOT__RXN07: now also U7.1 (A1); no longer U6.1 (A1)
- net GPIOT__RXN08: now also U6.7 (A5); no longer U4.7 (A5)
- net GPIOT__RXN09: now also U2.3 (A3); no longer U10.3 (A3)
- net GPIOT__RXN11: now also U8.3 (A3)
- net GPIOT__RXN12: now also U8.9 (A7)
- net GPIOT__RXN13: now also U8.2 (A2)
- net GPIOT__RXN14: now also U8.7 (A5)
- net GPIOT__RXN15: now also U2.9 (A7); no longer U10.9 (A7)
- net GPIOT__RXN16: now also U2.7 (A5); no longer U10.7 (A5)
- net GPIOT__RXN17: now also U2.2 (A2); no longer U10.2 (A2)
- net GPIOT__RXN18: now also U6.1 (A1); no longer U4.1 (A1)
- net GPIOT__RXN19: now also U7.9 (A7); no longer U6.9 (A7)
- net GPIOT__RXN20: now also U1.2 (A2); no longer U5.2 (A2)
- net GPIOT__RXN21: now also U6.4 (A4); no longer U4.4 (A4)
- net GPIOT__RXP01: now also U1.7 (A5); no longer U5.7 (A5)
- net GPIOT__RXP02: now also U7.8 (A6); no longer U6.8 (A6)
- net GPIOT__RXP03: now also U6.10 (A8); no longer U4.10 (A8)
- net GPIOT__RXP04: now also U7.4 (A4); no longer U6.4 (A4)
- net GPIOT__RXP05: now also U1.4 (A4); no longer U5.4 (A4)
- net GPIOT__RXP06: now also U1.10 (A8); no longer U5.10 (A8)
- net GPIOT__RXP07: now also U7.2 (A2); no longer U6.2 (A2)
- net GPIOT__RXP08: now also U6.8 (A6); no longer U4.8 (A6)
- net GPIOT__RXP09: now also U2.4 (A4); no longer U10.4 (A4)
- net GPIOT__RXP11: now also U8.4 (A4)
- net GPIOT__RXP12: now also U8.10 (A8)
- net GPIOT__RXP13: now also U8.1 (A1)
- net GPIOT__RXP14: now also U8.8 (A6)
- net GPIOT__RXP15: now also U2.10 (A8); no longer U10.10 (A8)
- net GPIOT__RXP16: now also U2.8 (A6); no longer U10.8 (A6)
- net GPIOT__RXP17: now also U2.1 (A1); no longer U10.1 (A1)
- net GPIOT__RXP18: now also U6.2 (A2); no longer U4.2 (A2)
- net GPIOT__RXP19: now also U7.10 (A8); no longer U6.10 (A8)
- net GPIOT__RXP20: now also U1.1 (A1); no longer U5.1 (A1)
- net GPIOT__RXP21: now also U6.3 (A3); no longer U4.3 (A3)
- net NETR20_2: now also U13.4 (PR)
- net NetR10_2: now also U10.6 (OE)
- net NetR1_2: now also U6.6 (OE); no longer U4.6 (OE)
- net NetR2_2: now also U1.6 (OE); no longer U5.6 (OE)
- net NetR3_2: now also U7.6 (OE); no longer U6.6 (OE)
- net NetR4_2: now also U2.6 (OE); no longer U10.6 (OE)
- net NetR5_2: now also U8.6 (OE)
- net NetR6_2: now also U3.6 (OE); no longer U7.6 (OE)
- net NetR7_2: now also U4.6 (OE); no longer U8.6 (OE)
- net NetR9_2: now also U5.6 (OE)
- net VCC5V: now also U13.6 (VIN2)
- net VCCB_1: now also U7.5 (VCCA); no longer U4.5 (VCCA)
- net VCCB_2: now also U1.5 (VCCA), U2.5 (VCCA); no longer U10.5 (VCCA), U5.5 (VCCA)
- net VCCB_3: now also U8.5 (VCCA)
- net VCCB_4: now also U4.5 (VCCA), U3.5 (VCCA); no longer U7.5 (VCCA), U8.5 (VCCA)
- net VCCB_5: now also U10.5 (VCCA), U5.5 (VCCA)
- net at R4.1: now also U13.8 (ST)
- net at J23.A5 (CC1): now also R19.1
- net at J23.B5 (CC2): now also R18.1
- no-connect marks 2 -> 0
