File: GPIO HAT 2/GPIO HAT 2/GPIO HAT 2.kicad_pcb (KiCad board)
At the start: 4 copper layers, 85 x 74.6 mm, 106 parts, among them J1 ., J10 ., J11 ., J12 ., J13 ., J14 ., J15 ., J16 ., J17 ., J18 ., J19 ., J2 ., J20 ., J21 LVDS, J22 LVDS, J23 USB_C_Receptacle_PowerOnly_6P, J24 02x02, J3 ., J4 ., J5 ., J6 ., J7 ., J8 ., J9 ., U1 TXB0108DQSR, U10 TXB0108DQSR, U11 SY8088IAAC, U12 SY8088IAAC, U13 TPS2117, U2 TXB0108DQSR, U3 TXB0108DQSR, U4 TXB0108DQSR, U5 TXB0108DQSR, U6 TXB0108DQSR, U7 TXB0108DQSR, U8 TXB0108DQSR, U9 TXB0108DQSR

Commit message: Gerber Generated
Parts:
- moved R5 0.47 mm to (169.8, 132.5)
- moved C11 0.17 mm to (169.2, 130.7)
- moved R3 0.13 mm to (168.7, 132.5)
