File: GPIO HAT 2/GPIO HAT 2.kicad_sch (KiCad schematic)
At the start: 101 parts, among them J1 ., J10 ., J11 ., J12 ., J13 ., J14 ., J15 ., J16 ., J17 ., J18 ., J19 ., J2 ., J20 ., J21 LVDS, J22 LVDS, J23 USB_C_Receptacle_PowerOnly_6P, J24 02x02, J3 ., J4 ., J5 ., J6 ., J7 ., J8 ., J9 ., U11 SY8088IAAC, U12 SY8088IAAC, U13 TPS2117

Commit message: Project file generated
BOM, HTML , PDFs
Parts:
- C1, C12, C13, C14, C16, C17, C18, C2, C3, C5, C6, C7, C8, C9: VOLTAGE 10V -> 25V
- C10, C11, C19, C20, C21, C23, C24, C25, C26, C27, C28, C29, C30, C31, C32, C33, C34, C35, C36, C37, C38: value 0.1uF -> 100nF; VOLTAGE 10V -> 25V
- C22: value 0.1uF -> 100nf; VOLTAGE 10V -> 25V
- J21, J22: Manufacturer_Part_Number DF40C-60DS-0.4V(51) -> DF40C-60DP-0.4V(51)
- R2: value 22.2K -> 22.1K
